File: hardware/DotDriver.kicad_pcb (KiCad board)
At the start: 2 copper layers, 90 x 66 mm, 50 parts, among them IC1 SY8120B1ABC, IC2 74HCT125D,653, IC3 74HCT125D,653, J1 USB_C_Receptacle_USB2.0_16P, J2 Conn_01x05_Pin, J3 Conn_01x02_Pin, J5 Conn_01x15, Q1 NPN, U1 ESP32-S3-WROOM-1, U2 LM2576HVS-5, U3 IRF4905S

Commit message: Added inductive kickback protection diode, fixed MOSFET drain/source mixup
Parts:
- added U4: FR207, lib:DO15-12, F.Cu at (96.2, 80.7)
- moved G*** 3.18 mm to (106.8, 86.4)
- moved G*** 3.09 mm to (98.5, 95.1)
Connections:
- U3 pad 2: V IN -> Power Pulse
- U3 pad 3: Power Pulse -> V IN
Routing:
- net Power Pulse: track 77.2 -> 106.6 mm
- net V IN: track 164.4 -> 186.0 mm
